File: Chiqoo2/Chiqoo2.brd (EAGLE design)
At the start: 82.5 x 47 mm, 46 parts, among them IC2 ADP1613, J1 POWER_JACKPTH, J2 M023.5MM, J3 M023.5MM, J6 M02PTH, U1 LT3652

Commit message: Chiqoo2 fixes
Parts:
- removed STANDOFF1, STANDOFF2, STANDOFF4: STAND-OFF, SparkFun-Electromechanical:STAND-OFF
- removed U$1: EG2315, bootstrapsolar:EG2315
- added SW1: EG2315, bootstrapsolar:EG2315
- C1, C2, C4: device adafruit:C025-025X050 -> adafruit:C050-024X044
- J2: value M023.5MM -> M02PTH; device SparkFun-Connectors:SCREWTERMINAL-3.5MM-2 -> SparkFun-Connectors:1X02
- X2: device con-berg:PN87520 -> bootstrapsolar:PN87520
- moved FID1 7.13 mm to (14.7, 3.05)
- moved J2 4.96 mm to (10.2, 4.45), turned to 180 degrees
- moved C1 2.69 mm to (12.1, 17.1)
- moved BATT1 1.91 mm to (41.3, 41.9)
- moved J1 1.91 mm to (-3.81, 26.0)
- moved C4 1.27 mm to (52.1, 17.1)
- moved C6 1.27 mm to (14.6, 9.78)
- moved LOGO2 1.27 mm to (14.7, 3.05)
- renumbered U1 to IC1
Connections:
- net +5V: now also SW1.2, SW1.6; no longer U$1.2, U$1.6
- net N$11: now also SW1.3, SW1.7; no longer U$1.3, U$1.7
- net N$14: now also SW1.4, SW1.8; no longer U$1.4, U$1.8
Routing:
- net V_BATT: track 56.8 -> 62.5 mm
- net VIN: track 33.6 -> 37.3 mm
- net N$14: track 32.2 -> 34.2 mm
- net N$11: track 16.4 -> 17.4 mm
- net TIMER: track 5.28 -> 4.31 mm
Other:
- outline, holes or cut-outs redrawn
- board text added: "Rev. 20140722"
- board text added: "http://solartothechildren.org"
- board text removed: "BootstrapSolar.com"
- board text removed: "Rev. 20140620"
- board text removed: "http://solar2thepeople.org"
