File: Chiqoo2/Chiqoo2.sch (EAGLE design)
At the start: 46 parts, among them IC2 ADP1613, J1 POWER_JACKPTH, J2 M023.5MM, J3 M023.5MM, J6 M02PTH, U1 LT3652

Commit message: Chiqoo2 fixes
Parts:
- removed STANDOFF1, STANDOFF2, STANDOFF4: STAND-OFF, SparkFun-Electromechanical:STAND-OFF
- C1, C2, C4: device adafruit:C-US025-025X050 -> adafruit:C-US050-024X044
- J2: value M023.5MM -> M02PTH; device SparkFun-Connectors:M023.5MM -> SparkFun-Connectors:M02PTH
- X2: device con-berg:PN87520 -> bootstrapsolar:PN87520
- renumbered U$1 to SW1, U1 to IC1
Changed lines of the file:
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@@
 <parts>
 <part name="FRAME1" library="SparkFun-Aesthetics" deviceset="FRAME-LETTER" device=""/>
-<part name="U1" library="bootstrapsolar" deviceset="LT3652" device="" value="LT3652"/>
+<part name="IC1" library="bootstrapsolar" deviceset="LT3652" device="" value="LT3652"/>
 <part name="R1" library="adafruit" deviceset="R-US_" device="0204/5" value="0.1"/>
-<part name="C1" library="adafruit" deviceset="C-US" device="025-025X050" value="10uF"/>
+<part name="C1" library="adafruit" deviceset="C-US" device="050-024X044" value="10uF"/>
 <part name="C3" library="adafruit" deviceset="CPOL-US" device="E5-5" value="100uF"/>
-<part name="C2" library="adafruit" deviceset="C-US" device="025-025X050" value="10uF"/>
+<part name="C2" library="adafruit" deviceset="C-US" device="050-024X044" value="10uF"/>
 <part name="L1" library="bootstrapsolar" deviceset="L-5MM-THRUHOLE" device="" value="68uH"/>
 <part name="D1" library="bootstrapsolar" deviceset="SCHOTTKY-DIODE" device="DIODE-5" value="1N5818"/>
@@
 <part name="SUPPLY4" library="SparkFun-Aesthetics" deviceset="VIN" device=""/>
 <part name="LOGO2" library="SparkFun-Aesthetics" deviceset="OSHW-LOGO" device="M"/>
-<part name="STANDOFF1" library="SparkFun-Electromechanical" deviceset="STAND-OFF" device=""/>
-<part name="STANDOFF2" library="SparkFun-Electromechanical" deviceset="STAND-OFF" device=""/>
-<part name="STANDOFF4" library="SparkFun-Electromechanical" deviceset="STAND-OFF" device=""/>
 <part name="R4" library="adafruit" deviceset="R-US_" device="0204/5" value="100"/>
 <part name="R5" library="adafruit" deviceset="R-US_" device="0204/5" value="100"/>
@@
 <part name="L3" library="bootstrapsolar" deviceset="L-5MM-THRUHOLE" device="" value="4.7uH"/>
 <part name="D4" library="bootstrapsolar" deviceset="SCHOTTKY-DIODE" device="" value="1N5820"/>
-<part name="C4" library="adafruit" deviceset="C-US" device="025-025X050" value="10uF"/>
+<part name="C4" library="adafruit" deviceset="C-US" device="050-024X044" value="10uF"/>
 <part name="C10" library="resistor" deviceset="C-US" device="050-024X044" value="33nF"/>
 <part name="C11" library="resistor" deviceset="C-US" device="025-025X050" value="1200pF"/>
-<part name="X2" library="con-berg" deviceset="PN87520" device=""/>
+<part name="X2" library="bootstrapsolar" deviceset="PN87520" device=""/>
 <part name="SUPPLY15" library="supply2" deviceset="GND" device=""/>
-<part name="J2" library="SparkFun-Connectors" deviceset="M02" device="3.5MM"/>
+<part name="J2" library="SparkFun-Connectors" deviceset="M02" device="PTH" value="M02PTH"/>
 <part name="R_THERM" library="adafruit" deviceset="R-US_" device="0204/5" value="10k"/>
 <part name="LED1" library="adafruit" deviceset="LED" device="3MM" value="GREEN"/>
 <part name="LED2" library="adafruit" deviceset="LED" device="3MM" value="RED"/>
-<part name="J3" library="SparkFun-Connectors" deviceset="M02" device="3.5MM"/>
-<part name="U$1" library="bootstrapsolar" deviceset="EG2315" device=""/>
+<part name="J3" library="SparkFun-Connectors" deviceset="M02" device="3.5MM" value="M023.5MM"/>
+<part name="SW1" library="bootstrapsolar" deviceset="EG2315" device=""/>
 <part name="GND6" library="SparkFun-Aesthetics" deviceset="GND" device=""/>
 <part name="LED3" library="adafruit" deviceset="LED" device="5MM" value="WHITE2"/>
@@
 <instance part="FRAME1" gate="G$1" x="0" y="0"/>
 <instance part="FRAME1" gate="G$2" x="147.32" y="0"/>
-<instance part="U1" gate="G$1" x="30.48" y="124.46"/>
+<instance part="IC1" gate="G$1" x="30.48" y="124.46"/>
 <instance part="R1" gate="G$1" x="104.14" y="152.4"/>
 <instance part="C1" gate="G$1" x="7.62" y="144.78"/>
@@
 <instance part="J6" gate="G$1" x="210.82" y="127" rot="R180"/>
 <instance part="GND5" gate="1" x="38.1" y="25.4"/>
-<instance part="SUPPLY4" gate="G$1" x="33.02" y="63.5"/>
+<instance part="SUPPLY4" gate="G$1" x="33.02" y="91.44"/>
 <instance part="LOGO2" gate="G$1" x="175.26" y="48.26"/>
-<instance part="STANDOFF1" gate="G$1" x="246.38" y="25.4"/>
-<instance part="STANDOFF2" gate="G$1" x="246.38" y="27.94"/>
-<instance part="STANDOFF4" gate="G$1" x="243.84" y="25.4"/>
 <instance part="R4" gate="G$1" x="180.34" y="167.64"/>
 <instance part="R5" gate="G$1" x="180.34" y="157.48"/>
@@
 <instance part="LED2" gate="G$1" x="190.5" y="157.48" rot="R90"/>
 <instance part="J3" gate="G$1" x="241.3" y="60.96" rot="R180"/>
-<instance part="U$1" gate="G$1" x="134.62" y="114.3" rot="R270"/>
+<instance part="SW1" gate="G$1" x="134.62" y="114.3" rot="R270"/>
 <instance part="GND6" gate="1" x="172.72" y="88.9"/>
 <instance part="LED3" gate="G$1" x="162.56" y="99.06" rot="R90"/>
@@
 <net name="SW" class="0">
 <segment>
-<pinref part="U1" gate="G$1" pin="SW"/>
+<pinref part="IC1" gate="G$1" pin="SW"/>
 <pinref part="L1" gate="G$1" pin="1"/>
 <pinref part="C5" gate="G$1" pin="2"/>
@@
 <net name="SENSE" class="0">
 <segment>
-<pinref part="U1" gate="G$1" pin="SENSE"/>
+<pinref part="IC1" gate="G$1" pin="SENSE"/>
 <wire x1="60.96" y1="142.24" x2="96.52" y2="142.24" width="0.1524" layer="91"/>
 <wire x1="96.52" y1="142.24" x2="96.52" y2="152.4" width="0.1524" layer="91"/>
@@
 <segment>
 <pinref part="C1" gate="G$1" pin="1"/>
-<pinref part="U1" gate="G$1" pin="VIN"/>
+<pinref part="IC1" gate="G$1" pin="VIN"/>
 <wire x1="22.86" y1="152.4" x2="25.4" y2="152.4" width="0.1524" layer="91"/>
-<pinref part="U1" gate="G$1" pin="VIN_REG"/>
+<pinref part="IC1" gate="G$1" pin="VIN_REG"/>
 <wire x1="25.4" y1="147.32" x2="22.86" y2="147.32" width="0.1524" layer="91"/>
 <wire x1="22.86" y1="147.32" x2="22.86" y2="152.4" width="0.1524" layer="91"/>
 <junction x="22.86" y="152.4"/>
 <wire x1="17.78" y1="152.4" x2="22.86" y2="152.4" width="0.1524" layer="91"/>
-<pinref part="U1" gate="G$1" pin="!SHDN"/>
+<pinref part="IC1" gate="G$1" pin="!SHDN"/>
 <wire x1="25.4" y1="142.24" x2="17.78" y2="142.24" width="0.1524" layer="91"/>
 <wire x1="17.78" y1="142.24" x2="17.78" y2="152.4" width="0.1524" layer="91"/>
@@
 </segment>
 <segment>
-<wire x1="33.02" y1="63.5" x2="33.02" y2="53.34" width="0.1524" layer="91"/>
 <pinref part="SUPPLY4" gate="G$1" pin="VIN"/>
+<wire x1="33.02" y1="91.44" x2="33.02" y2="53.34" width="0.1524" layer="91"/>
 <wire x1="33.02" y1="53.34" x2="33.02" y2="38.1" width="0.1524" layer="91"/>
 <wire x1="20.32" y1="38.1" x2="33.02" y2="38.1" width="0.1524" layer="91"/>
@@
 </segment>
 <segment>
-<pinref part="U1" gate="G$1" pin="GND_PAD"/>
+<pinref part="IC1" gate="G$1" pin="GND_PAD"/>
 <pinref part="C6" gate="G$1" pin="1"/>
 <wire x1="43.18" y1="106.68" x2="43.18" y2="121.92" width="0.1524" layer="91"/>
@@
 <segment>
 <pinref part="C5" gate="G$1" pin="1"/>
-<pinref part="U1" gate="G$1" pin="BOOST"/>
+<pinref part="IC1" gate="G$1" pin="BOOST"/>
 <wire x1="68.58" y1="147.32" x2="63.5" y2="147.32" width="0.1524" layer="91"/>
 <pinref part="D2" gate="G$1" pin="C"/>
@@
 <segment>
 <pinref part="C6" gate="G$1" pin="2"/>
-<pinref part="U1" gate="G$1" pin="TIMER"/>
+<pinref part="IC1" gate="G$1" pin="TIMER"/>
 <wire x1="22.86" y1="127" x2="25.4" y2="127" width="0.1524" layer="91"/>
 </segment>
@@
 <junction x="78.74" y="121.92"/>
 <wire x1="63.5" y1="121.92" x2="63.5" y2="127" width="0.1524" layer="91"/>
-<pinref part="U1" gate="G$1" pin="VFB"/>
+<pinref part="IC1" gate="G$1" pin="VFB"/>
 <wire x1="63.5" y1="127" x2="60.96" y2="127" width="0.1524" layer="91"/>
 <wire x1="63.5" y1="121.92" x2="78.74" y2="121.92" width="0.1524" layer="91"/>
@@
 <net name="!CHRG" class="0">
 <segment>
-<pinref part="U1" gate="G$1" pin="!CHRG"/>
+<pinref part="IC1" gate="G$1" pin="!CHRG"/>
 <wire x1="25.4" y1="137.16" x2="22.86" y2="137.16" width="0.1524" layer="91"/>
 <label x="22.86" y="137.16" size="1.778" layer="95" rot="R180" xref="yes"/>
@@
 <net name="!FAULT" class="0">
 <segment>
-<pinref part="U1" gate="G$1" pin="!FAULT"/>
+<pinref part="IC1" gate="G$1" pin="!FAULT"/>
 <wire x1="25.4" y1="132.08" x2="22.86" y2="132.08" width="0.1524" layer="91"/>
 <label x="22.86" y="132.08" size="1.778" layer="95" rot="R180" xref="yes"/>
@@
 <pinref part="R1" gate="G$1" pin="2"/>
 <wire x1="109.22" y1="152.4" x2="111.76" y2="152.4" width="0.1524" layer="91"/>
-<pinref part="U1" gate="G$1" pin="BAT"/>
+<pinref part="IC1" gate="G$1" pin="BAT"/>
 <wire x1="60.96" y1="137.16" x2="78.74" y2="137.16" width="0.1524" layer="91"/>
 <wire x1="78.74" y1="137.16" x2="111.76" y2="137.16" width="0.1524" layer="91"/>
@@
 </segment>
 <segment>
-<pinref part="U$1" gate="G$1" pin="2"/>
+<pinref part="SW1" gate="G$1" pin="2"/>
 <wire x1="142.24" y1="116.84" x2="147.32" y2="116.84" width="0.1524" layer="91"/>
 <wire x1="147.32" y1="116.84" x2="147.32" y2="127" width="0.1524" layer="91"/>
@@
 <net name="N$2" class="0">
 <segment>
-<pinref part="U1" gate="G$1" pin="NTC"/>
+<pinref part="IC1" gate="G$1" pin="NTC"/>
 <pinref part="R_THERM" gate="G$1" pin="1"/>
 </segment>
@@
 <net name="N$11" class="0">
 <segment>
-<pinref part="U$1" gate="G$1" pin="3"/>
+<pinref part="SW1" gate="G$1" pin="3"/>
 <pinref part="R6" gate="G$1" pin="1"/>
 <wire x1="142.24" y1="114.3" x2="147.32" y2="114.3" width="0.1524" layer="91"/>
@@
 <pinref part="R10" gate="G$1" pin="1"/>
 <wire x1="147.32" y1="99.06" x2="149.86" y2="99.06" width="0.1524" layer="91"/>
-<pinref part="U$1" gate="G$1" pin="4"/>
+<pinref part="SW1" gate="G$1" pin="4"/>
 <wire x1="142.24" y1="111.76" x2="142.24" y2="99.06" width="0.1524" layer="91"/>
 <wire x1="142.24" y1="99.06" x2="147.32" y2="99.06" width="0.1524" layer="91"/>
